Commit message: description update

File: manipulator_x_description/urdf/manipulator_x_4dof.xacro (robot description, xacro)
@@ -257,11 +257,11 @@
       <origin xyz="0 0 0" rpy="0 0 0"/>
       <geometry>
-        <mesh filename="package://manipulator_x_description/meshes/manipulator_x_link9.stl" scale="0.001 0.001 0.001"/>
-      </geometry>
-    </collision>
-    <visual>
-      <origin xyz="0 0 0" rpy="0 0 0"/>
-      <geometry>
-        <mesh filename="package://manipulator_x_description/meshes/manipulator_x_link9.stl" scale="0.001 0.001 0.001"/>
+        <mesh filename="package://manipulator_x_description/meshes/manipulator_x_link_grip1.stl" scale="0.001 0.001 0.001"/>
+      </geometry>
+    </collision>
+    <visual>
+      <origin xyz="0 0 0" rpy="0 0 0"/>
+      <geometry>
+        <mesh filename="package://manipulator_x_description/meshes/manipulator_x_link_grip1.stl" scale="0.001 0.001 0.001"/>
       </geometry>
       <material name="grey"/>
@@ -298,11 +298,11 @@
       <origin xyz="0 0 0" rpy="0 0 0"/>
       <geometry>
-        <mesh filename="package://manipulator_x_description/meshes/manipulator_x_link8.stl" scale="0.001 0.001 0.001"/>
-      </geometry>
-    </collision>
-    <visual>
-      <origin xyz="0 0 0" rpy="0 0 0"/>
-      <geometry>
-        <mesh filename="package://manipulator_x_description/meshes/manipulator_x_link8.stl" scale="0.001 0.001 0.001"/>
+        <mesh filename="package://manipulator_x_description/meshes/manipulator_x_link_grip2.stl" scale="0.001 0.001 0.001"/>
+      </geometry>
+    </collision>
+    <visual>
+      <origin xyz="0 0 0" rpy="0 0 0"/>
+      <geometry>
+        <mesh filename="package://manipulator_x_description/meshes/manipulator_x_link_grip2.stl" scale="0.001 0.001 0.001"/>
       </geometry>
       <material name="grey"/>

Commit message: update manipulator-x4 urdf

File: manipulator_x_description/urdf/manipulator_x_4dof.xacro (robot description, xacro)
@@ -62,10 +62,11 @@
       <material name="grey"/>
     </visual>
-    <inertial>
+<!--    <inertial>
       <origin xyz="0.00025 0.00000 0.01780" rpy="0 0 0"/>
       <mass value="0.087"/>
       <inertia ixx="1.0" ixy="0.0" ixz="0.0" iyy="1.0" iyz="0.0" izz="1.0" />
-      <!--<inertia ixx="0.00001378" ixy="0.0" ixz="-0.00000025" iyy="0.00002381" iyz="0.0" izz="0.00002107" />-->
-    </inertial>
+      <inertia ixx="0.00001378" ixy="0.0" ixz="-0.00000025" iyy="0.00002381" iyz="0.0" izz="0.00002107" />
+    </inertial>
+-->
   </link>
   <!-- Joint 1 -->
@@ -103,10 +104,11 @@
       <material name="grey"/>
     </visual>
-    <inertial>
+<!--    <inertial>
       <origin xyz="0.00002 -0.00045 0.03293" rpy="0 0 0"/>
       <mass value="0.117"/>
       <inertia ixx="1.0" ixy="0.0" ixz="0.0" iyy="1.0" iyz="0.0" izz="1.0" />
-      <!--<inertia ixx="0.00004110" ixy="0.0" ixz="-0.00000025" iyy="0.00002381" iyz="0.0" izz="0.00002107" />-->
-    </inertial>
+      <inertia ixx="0.00004110" ixy="0.0" ixz="-0.00000025" iyy="0.00002381" iyz="0.0" izz="0.00002107" />
+    </inertial>
+-->
   </link>
   <!-- Joint 2 -->
@@ -132,5 +134,5 @@
   <link name="link3">
     <collision>
-      <origin xyz="0 0 0" rpy="0 0 0"/>
+      <origin xyz="0 -0.020 0" rpy="0 0 0"/>
       <geometry>
         <mesh filename="package://manipulator_x_description/meshes/manipulator_x_link3.stl" scale="0.001 0.001 0.001"/>
@@ -138,5 +140,5 @@
     </collision>
     <visual>
-      <origin xyz="0 0 0" rpy="0 0 0"/>
+      <origin xyz="0 -0.020 0" rpy="0 0 0"/>
       <geometry>
         <mesh filename="package://manipulator_x_description/meshes/manipulator_x_link3.stl" scale="0.001 0.001 0.001"/>
@@ -144,10 +146,11 @@
       <material name="grey"/>
     </visual>
-    <inertial>
+<!--    <inertial>
       <origin xyz="0.00966 -0.00034 0.11795" rpy="0 0 0"/>
       <mass value="0.156"/>
       <inertia ixx="1.0" ixy="0.0" ixz="0.0" iyy="1.0" iyz="0.0" izz="1.0" />
-      <!--<inertia ixx="0.00041624" ixy="0.00000017" ixz="-0.00004492" iyy="0.00042758" iyz="0.00000159" izz="0.00005317" />-->
-    </inertial>
+      <inertia ixx="0.00041624" ixy="0.00000017" ixz="-0.00004492" iyy="0.00042758" iyz="0.00000159" izz="0.00005317" />
+    </inertial>
+-->
   </link>
   <!-- Joint 3 -->
@@ -155,5 +158,5 @@
     <parent link="link3"/>
     <child link="link4"/>
-    <origin xyz="0.024 0.0 0.14815" rpy="0 0 0"/>
+    <origin xyz="0.024 0.0 0.12165" rpy="0 0 0"/>
     <axis xyz="0 -1 0"/>
     <limit velocity="6.5" effort="1000" lower="${-pi*0.5}" upper="${pi*0.5}" />
@@ -173,5 +176,5 @@
   <link name="link4">
     <collision>
-      <origin xyz="0 0 0" rpy="0 0 0"/>
+      <origin xyz="0 -0.020 0.0" rpy="0 0 0"/>
       <geometry>
         <mesh filename="package://manipulator_x_description/meshes/manipulator_x_link4.stl" scale="0.001 0.001 0.001"/>
@@ -179,5 +182,5 @@
     </collision>
     <visual>
-      <origin xyz="0 0 0" rpy="0 0 0"/>
+      <origin xyz="0 -0.020 0.0" rpy="0 0 0"/>
       <geometry>
         <mesh filename="package://manipulator_x_description/meshes/manipulator_x_link4.stl" scale="0.001 0.001 0.001"/>
@@ -185,10 +188,11 @@
       <material name="grey"/>
     </visual>
-    <inertial>
+<!--    <inertial>
       <origin xyz="0.11076 -0.00035 0.00050" rpy="0 0 0"/>
       <mass value="0.149"/>
       <inertia ixx="1.0" ixy="0.0" ixz="0.0" iyy="1.0" iyz="0.0" izz="1.0" />
-      <!--<inertia ixx="0.00003083" ixy="0.00000147" ixz="-0.00000222" iyy="0.00036703" iyz="-0.00000003" izz="0.00037667" />-->
-    </inertial>
+      <inertia ixx="0.00003083" ixy="0.00000147" ixz="-0.00000222" iyy="0.00036703" iyz="-0.00000003" izz="0.00037667" />
+    </inertial>
+-->
   </link>
   <!-- Joint 4 -->
@@ -196,5 +200,5 @@
     <parent link="link4"/>
     <child link="link5"/>
-    <origin xyz="0.15 0.0 0.0" rpy="0 0 0"/>
+    <origin xyz="0.1235 0.0 0.0" rpy="0 0 0"/>
     <axis xyz="0 -1 0"/>
     <limit velocity="6.5" effort="1000" lower="${-pi*0.5}" upper="${pi*0.5}" />
@@ -214,5 +218,5 @@
   <link name="link5">
     <collision>
-      <origin xyz="0 0 0" rpy="0 0 0"/>
+      <origin xyz="0 -0.020 0" rpy="0 0 0"/>
       <geometry>
         <mesh filename="package://manipulator_x_description/meshes/manipulator_x_link5.stl" scale="0.001 0.001 0.001"/>
@@ -220,5 +224,5 @@
     </collision>
     <visual>
-      <origin xyz="0 0 0" rpy="0 0 0"/>
+      <origin xyz="0 -0.020 0" rpy="0 0 0"/>
       <geometry>
         <mesh filename="package://manipulator_x_description/meshes/manipulator_x_link5.stl" scale="0.001 0.001 0.001"/>
@@ -226,18 +230,19 @@
       <material name="grey"/>
     </visual>
-    <inertial>
+<!--    <inertial>
       <origin xyz="0.03767 0.00262 -0.00043" rpy="0 0 0"/>
       <mass value="0.124"/>
       <inertia ixx="1.0" ixy="0.0" ixz="0.0" iyy="1.0" iyz="0.0" izz="1.0" />
-      <!--<inertia ixx="0.00004822" ixy="-0.00000148" ixz="0.00000024" iyy="0.00004342" iyz="0.00000014" izz="0.00005784" />-->
-    </inertial>
+      <inertia ixx="0.00004822" ixy="-0.00000148" ixz="0.00000024" iyy="0.00004342" iyz="0.00000014" izz="0.00005784" />
+    </inertial>
+-->
   </link>
   <!-- Grip Joint -->
-  <joint name="grip_joint" type="revolute">
+  <joint name="grip_joint" type="prismatic">
     <parent link="link5"/>
     <child link="grip_link"/>
-    <origin xyz="0.04225 -0.01600 0.02300" rpy="0 0 0"/>
-    <axis xyz="0 0 1"/>
-    <limit velocity="6.5" effort="1000" lower="${-0.5*pi}" upper="${0.5*pi}" />
+    <origin xyz="0.0982 -0.036 0.0" rpy="0 0 0"/>
+    <axis xyz="1 0 0"/>
+    <limit velocity="6.5" effort="1000" lower="${0.0}" upper="${0.025}" />
     <dynamics damping="0.7"/>
   </joint>
@@ -255,5 +260,5 @@
   <link name="grip_link">
     <collision>
-      <origin xyz="0 0 0" rpy="0 0 0"/>
+      <origin xyz="-0.0982 0.016 0" rpy="0 0 0"/>
       <geometry>
         <mesh filename="package://manipulator_x_description/meshes/manipulator_x_link_grip1.stl" scale="0.001 0.001 0.001"/>
@@ -261,5 +266,5 @@
     </collision>
     <visual>
-      <origin xyz="0 0 0" rpy="0 0 0"/>
+      <origin xyz="-0.0982 0.016 0" rpy="0 0 0"/>
       <geometry>
         <mesh filename="package://manipulator_x_description/meshes/manipulator_x_link_grip1.stl" scale="0.001 0.001 0.001"/>
@@ -267,18 +272,19 @@
       <material name="grey"/>
     </visual>
-    <inertial>
+<!--    <inertial>
       <origin xyz="0.02666 -0.00910 -0.02300" rpy="0 0 0"/>
       <mass value="0.06721"/>
       <inertia ixx="1.0" ixy="0.0" ixz="0.0" iyy="1.0" iyz="0.0" izz="1.0" />
-      <!--<inertia ixx="0.00002875" ixy="-0.00000593" ixz="-0.00000006" iyy="0.00006646" iyz="-0.00000009" izz="0.00005474" />-->
-    </inertial>
+      <inertia ixx="0.00002875" ixy="-0.00000593" ixz="-0.00000006" iyy="0.00006646" iyz="-0.00000009" izz="0.00005474" />
+    </inertial>
+-->
   </link>
   <!-- Grip Joint Sub -->
-  <joint name="grip_joint_sub" type="revolute">
+  <joint name="grip_joint_sub" type="prismatic">
     <parent link="link5"/>
     <child link="grip_link_sub"/>
-    <origin xyz="0.04225 0.01600 0.02300" rpy="0 0 0"/>
-    <axis xyz="0 0 -1"/>
-    <limit velocity="6.5" effort="1000" lower="${-0.5*pi}" upper="${0.5*pi}" />
+    <origin xyz="0.0982 0.036 0" rpy="0 0 0"/>
+    <axis xyz="1 0 0"/>
+    <limit velocity="6.5" effort="1000" lower="${0.0}" upper="${0.025}" />
     <dynamics damping="0.7"/>
   </joint>
@@ -296,5 +302,5 @@
   <link name="grip_link_sub">
     <collision>
-      <origin xyz="0 0 0" rpy="0 0 0"/>
+      <origin xyz="-0.0982 -0.056 0" rpy="0 0 0"/>
       <geometry>
         <mesh filename="package://manipulator_x_description/meshes/manipulator_x_link_grip2.stl" scale="0.001 0.001 0.001"/>
@@ -302,5 +308,5 @@
     </collision>
     <visual>
-      <origin xyz="0 0 0" rpy="0 0 0"/>
+      <origin xyz="-0.0982 -0.056 0" rpy="0 0 0"/>
       <geometry>
         <mesh filename="package://manipulator_x_description/meshes/manipulator_x_link_grip2.stl" scale="0.001 0.001 0.001"/>
@@ -308,10 +314,11 @@
       <material name="grey"/>
     </visual>
-    <inertial>
+<!--    <inertial>
       <origin xyz="0.02666 0.00910 -0.02300" rpy="0 0 0"/>
       <mass value="0.06721"/>
       <inertia ixx="1.0" ixy="0.0" ixz="0.0" iyy="1.0" iyz="0.0" izz="1.0" />
-      <!--<inertia ixx="0.00002875" ixy="0.00000593" ixz="0.00000006" iyy="0.00006646" iyz="-0.00000009" izz="0.00005474" />-->
-    </inertial>
+      <inertia ixx="0.00002875" ixy="0.00000593" ixz="0.00000006" iyy="0.00006646" iyz="-0.00000009" izz="0.00005474" />
+    </inertial>
+-->
   </link>
 </robot>

Commit message: add gripper module

File: manipulator_x_description/urdf/manipulator_x_4dof.xacro (robot description, xacro)
@@ -242,7 +242,7 @@
     <parent link="link5"/>
     <child link="grip_link"/>
-    <origin xyz="0.0982 -0.036 0.0" rpy="0 0 0"/>
-    <axis xyz="1 0 0"/>
-    <limit velocity="6.5" effort="1000" lower="${0.0}" upper="${0.025}" />
+    <origin xyz="0.064 0.0 0.0" rpy="0 0 0"/>
+    <axis xyz="0 1 0"/>
+    <limit velocity="6.5" effort="1000" lower="0.0" upper="0.0" />
     <dynamics damping="0.7"/>
   </joint>
@@ -260,5 +260,5 @@
   <link name="grip_link">
     <collision>
-      <origin xyz="-0.0982 0.016 0" rpy="0 0 0"/>
+      <origin xyz="-0.064 -0.020 0" rpy="0 0 0"/>
       <geometry>
         <mesh filename="package://manipulator_x_description/meshes/manipulator_x_link_grip1.stl" scale="0.001 0.001 0.001"/>
@@ -266,5 +266,5 @@
     </collision>
     <visual>
-      <origin xyz="-0.0982 0.016 0" rpy="0 0 0"/>
+      <origin xyz="-0.064 -0.020 0" rpy="0 0 0"/>
       <geometry>
         <mesh filename="package://manipulator_x_description/meshes/manipulator_x_link_grip1.stl" scale="0.001 0.001 0.001"/>
@@ -284,7 +284,7 @@
     <parent link="link5"/>
     <child link="grip_link_sub"/>
-    <origin xyz="0.0982 0.036 0" rpy="0 0 0"/>
-    <axis xyz="1 0 0"/>
-    <limit velocity="6.5" effort="1000" lower="${0.0}" upper="${0.025}" />
+    <origin xyz="0.064 0.0 0" rpy="0 0 0"/>
+    <axis xyz="0 -1 0"/>
+    <limit velocity="6.5" effort="1000" lower="0.0" upper="0.0" />
     <dynamics damping="0.7"/>
   </joint>
@@ -302,5 +302,5 @@
   <link name="grip_link_sub">
     <collision>
-      <origin xyz="-0.0982 -0.056 0" rpy="0 0 0"/>
+      <origin xyz="-0.064 -0.020 0" rpy="0 0 0"/>
       <geometry>
         <mesh filename="package://manipulator_x_description/meshes/manipulator_x_link_grip2.stl" scale="0.001 0.001 0.001"/>
@@ -308,5 +308,5 @@
     </collision>
     <visual>
-      <origin xyz="-0.0982 -0.056 0" rpy="0 0 0"/>
+      <origin xyz="-0.064 -0.020 0" rpy="0 0 0"/>
       <geometry>
         <mesh filename="package://manipulator_x_description/meshes/manipulator_x_link_grip2.stl" scale="0.001 0.001 0.001"/>

Commit message: update urdf

File: manipulator_x_description/urdf/manipulator_x_4dof.xacro (robot description, xacro)
@@ -77,5 +77,5 @@
     <axis xyz="0 0 1"/>
     <limit velocity="6.5" effort="1000" lower="${-pi*0.9}" upper="${pi*0.9}" />
-    <dynamics damping="0.7"/>
+    <dynamics damping="0.1"/>
   </joint>
   <transmission name="tran1">
@@ -119,5 +119,5 @@
     <axis xyz="0 -1 0"/>
     <limit velocity="6.5" effort="1000" lower="${-pi*0.5}" upper="${pi*0.5}" />
-    <dynamics damping="0.7"/>
+    <dynamics damping="0.1"/>
   </joint>
   <transmission name="tran2">
@@ -161,5 +161,5 @@
     <axis xyz="0 -1 0"/>
     <limit velocity="6.5" effort="1000" lower="${-pi*0.5}" upper="${pi*0.5}" />
-    <dynamics damping="0.7"/>
+    <dynamics damping="0.1"/>
   </joint>
   <transmission name="tran3">
@@ -203,5 +203,5 @@
     <axis xyz="0 -1 0"/>
     <limit velocity="6.5" effort="1000" lower="${-pi*0.5}" upper="${pi*0.5}" />
-    <dynamics damping="0.7"/>
+    <dynamics damping="0.1"/>
   </joint>
   <transmission name="tran4">
@@ -244,6 +244,6 @@
     <origin xyz="0.064 0.0 0.0" rpy="0 0 0"/>
     <axis xyz="0 1 0"/>
-    <limit velocity="6.5" effort="1000" lower="0.0" upper="0.0" />
-    <dynamics damping="0.7"/>
+    <limit velocity="6.5" effort="1000" lower="-0.01" upper="0.035" />
+    <dynamics damping="0.1"/>
   </joint>
   <transmission name="tran7">
@@ -286,6 +286,6 @@
     <origin xyz="0.064 0.0 0" rpy="0 0 0"/>
     <axis xyz="0 -1 0"/>
-    <limit velocity="6.5" effort="1000" lower="0.0" upper="0.0" />
-    <dynamics damping="0.7"/>
+    <limit velocity="6.5" effort="1000" lower="-0.01" upper="0.035" />
+    <dynamics damping="0.1"/>
   </joint>
   <transmission name="tran8">

Commit message: update manipulator description

File: manipulator_x_description/urdf/manipulator_x_4dof.xacro (robot description, xacro)
@@ -1,5 +1,5 @@
 <?xml version="1.0"?>
 <!-- ROBOTIS Manipulator-X4 -->
-<robot name="/robotis/manipulator_x4" xmlns:xacro="http://www.ros.org/wiki/xacro">
+<robot name="/gazebo/robotis/manipulator_x4" xmlns:xacro="http://www.ros.org/wiki/xacro">
   <!-- some parameters -->
   <xacro:property name="pi" value="3.141592654" />
@@ -62,5 +62,5 @@
       <material name="grey"/>
     </visual>
-<!--    <inertial>
+    <inertial>
       <origin xyz="0.00025 0.00000 0.01780" rpy="0 0 0"/>
       <mass value="0.087"/>
@@ -68,5 +68,4 @@
       <inertia ixx="0.00001378" ixy="0.0" ixz="-0.00000025" iyy="0.00002381" iyz="0.0" izz="0.00002107" />
     </inertial>
--->
   </link>
   <!-- Joint 1 -->
@@ -82,8 +81,8 @@
     <type>transmission_interface/SimpleTransmission</type>
     <joint name="joint1">
-      <hardwareInterface>EffortJointInterface</hardwareInterface>
+      <hardwareInterface>PositionJointInterface</hardwareInterface>
     </joint>
     <actuator name="motor1">
-      <hardwareInterface>EffortJointInterface</hardwareInterface>
+      <hardwareInterface>PositionJointInterface</hardwareInterface>
       <mechanicalReduction>1</mechanicalReduction>
     </actuator>
@@ -104,5 +103,5 @@
       <material name="grey"/>
     </visual>
-<!--    <inertial>
+    <inertial>
       <origin xyz="0.00002 -0.00045 0.03293" rpy="0 0 0"/>
       <mass value="0.117"/>
@@ -110,5 +109,4 @@
       <inertia ixx="0.00004110" ixy="0.0" ixz="-0.00000025" iyy="0.00002381" iyz="0.0" izz="0.00002107" />
     </inertial>
--->
   </link>
   <!-- Joint 2 -->
@@ -124,8 +122,8 @@
     <type>transmission_interface/SimpleTransmission</type>
     <joint name="joint2">
-      <hardwareInterface>EffortJointInterface</hardwareInterface>
+      <hardwareInterface>PositionJointInterface</hardwareInterface>
     </joint>
     <actuator name="motor2">
-      <hardwareInterface>EffortJointInterface</hardwareInterface>
+      <hardwareInterface>PositionJointInterface</hardwareInterface>
       <mechanicalReduction>1</mechanicalReduction>
     </actuator>
@@ -146,5 +144,5 @@
       <material name="grey"/>
     </visual>
-<!--    <inertial>
+    <inertial>
       <origin xyz="0.00966 -0.00034 0.11795" rpy="0 0 0"/>
       <mass value="0.156"/>
@@ -152,5 +150,4 @@
       <inertia ixx="0.00041624" ixy="0.00000017" ixz="-0.00004492" iyy="0.00042758" iyz="0.00000159" izz="0.00005317" />
     </inertial>
--->
   </link>
   <!-- Joint 3 -->
@@ -166,8 +163,8 @@
     <type>transmission_interface/SimpleTransmission</type>
     <joint name="joint3">
-      <hardwareInterface>EffortJointInterface</hardwareInterface>
+      <hardwareInterface>PositionJointInterface</hardwareInterface>
     </joint>
     <actuator name="motor3">
-      <hardwareInterface>EffortJointInterface</hardwareInterface>
+      <hardwareInterface>PositionJointInterface</hardwareInterface>
       <mechanicalReduction>1</mechanicalReduction>
     </actuator>
@@ -188,5 +185,5 @@
       <material name="grey"/>
     </visual>
-<!--    <inertial>
+    <inertial>
       <origin xyz="0.11076 -0.00035 0.00050" rpy="0 0 0"/>
       <mass value="0.149"/>
@@ -194,5 +191,4 @@
       <inertia ixx="0.00003083" ixy="0.00000147" ixz="-0.00000222" iyy="0.00036703" iyz="-0.00000003" izz="0.00037667" />
     </inertial>
--->
   </link>
   <!-- Joint 4 -->
@@ -208,8 +204,8 @@
     <type>transmission_interface/SimpleTransmission</type>
     <joint name="joint4">
-      <hardwareInterface>EffortJointInterface</hardwareInterface>
+      <hardwareInterface>PositionJointInterface</hardwareInterface>
     </joint>
     <actuator name="motor4">
-      <hardwareInterface>EffortJointInterface</hardwareInterface>
+      <hardwareInterface>PositionJointInterface</hardwareInterface>
       <mechanicalReduction>1</mechanicalReduction>
     </actuator>
@@ -230,5 +226,5 @@
       <material name="grey"/>
     </visual>
-<!--    <inertial>
+    <inertial>
       <origin xyz="0.03767 0.00262 -0.00043" rpy="0 0 0"/>
       <mass value="0.124"/>
@@ -236,5 +232,4 @@
       <inertia ixx="0.00004822" ixy="-0.00000148" ixz="0.00000024" iyy="0.00004342" iyz="0.00000014" izz="0.00005784" />
     </inertial>
--->
   </link>
   <!-- Grip Joint -->
@@ -250,8 +245,8 @@
     <type>transmission_interface/SimpleTransmission</type>
     <joint name="grip_joint">
-      <hardwareInterface>EffortJointInterface</hardwareInterface>
+      <hardwareInterface>PositionJointInterface</hardwareInterface>
     </joint>
     <actuator name="motor7">
-      <hardwareInterface>EffortJointInterface</hardwareInterface>
+      <hardwareInterface>PositionJointInterface</hardwareInterface>
       <mechanicalReduction>1</mechanicalReduction>
     </actuator>
@@ -272,5 +267,5 @@
       <material name="grey"/>
     </visual>
-<!--    <inertial>
+    <inertial>
       <origin xyz="0.02666 -0.00910 -0.02300" rpy="0 0 0"/>
       <mass value="0.06721"/>
@@ -278,5 +273,4 @@
       <inertia ixx="0.00002875" ixy="-0.00000593" ixz="-0.00000006" iyy="0.00006646" iyz="-0.00000009" izz="0.00005474" />
     </inertial>
--->
   </link>
   <!-- Grip Joint Sub -->
@@ -292,8 +286,8 @@
     <type>transmission_interface/SimpleTransmission</type>
     <joint name="grip_joint_sub">
-      <hardwareInterface>EffortJointInterface</hardwareInterface>
+      <hardwareInterface>PositionJointInterface</hardwareInterface>
     </joint>
     <actuator name="motor8">
-      <hardwareInterface>EffortJointInterface</hardwareInterface>
+      <hardwareInterface>PositionJointInterface</hardwareInterface>
       <mechanicalReduction>1</mechanicalReduction>
     </actuator>
@@ -314,5 +308,5 @@
       <material name="grey"/>
     </visual>
-<!--    <inertial>
+    <inertial>
       <origin xyz="0.02666 0.00910 -0.02300" rpy="0 0 0"/>
       <mass value="0.06721"/>
@@ -320,5 +314,4 @@
       <inertia ixx="0.00002875" ixy="0.00000593" ixz="0.00000006" iyy="0.00006646" iyz="-0.00000009" izz="0.00005474" />
     </inertial>
--->
   </link>
 </robot>

Commit message: update xacro file

File: manipulator_x_description/urdf/manipulator_x_4dof.xacro (robot description, xacro)
@@ -15,19 +15,18 @@
     <origin xyz="0 0 0" rpy="0 0 0"/>
     <parent link="world"/>
-    <child link="link1"/>
+    <child link="base"/>
   </joint>
   <!-- Base Plate -->
-<!--
   <link name="base">
     <collision>
       <origin xyz="0 0 0" rpy="0 0 0"/>
       <geometry>
-        <mesh filename="package://manipulator_x_description/meshes/manipulator_x_base.stl" scale="0.001 0.001 0.001"/>
-      </geometry>
-    </collision>
-    <visual>
-      <origin xyz="0 0 0" rpy="0 0 0"/>
-      <geometry>
-        <mesh filename="package://manipulator_x_description/meshes/manipulator_x_base.stl" scale="0.001 0.001 0.001"/>
+        <mesh filename="package://manipulator_x_description/meshes/turtlebot3_premium.stl" scale="0.001 0.001 0.001"/>
+      </geometry>
+    </collision>
+    <visual>
+      <origin xyz="0 0 0" rpy="0 0 0"/>
+      <geometry>
+        <mesh filename="package://manipulator_x_description/meshes/turtlebot3_premium.stl" scale="0.001 0.001 0.001"/>
       </geometry>
       <material name="grey"/>
@@ -39,16 +38,13 @@
     </inertial>
   </link>
--->
   <!-- Base fixed joint -->
-<!--
   <joint name="base_fixed" type="fixed">
     <parent link="base"/>
     <child link="link1"/>
   </joint>
--->
   <!-- Link 1 -->
   <link name="link1">
     <collision>
-      <origin xyz="0 0 0" rpy="0 0 0"/>
+      <origin xyz="0.036 0 0.103" rpy="0 0 0"/>
       <geometry>
         <mesh filename="package://manipulator_x_description/meshes/manipulator_x_link1.stl" scale="0.001 0.001 0.001"/>
@@ -56,5 +52,5 @@
     </collision>
     <visual>
-      <origin xyz="0 0 0" rpy="0 0 0"/>
+      <origin xyz="0.036 0 0.103" rpy="0 0 0"/>
       <geometry>
         <mesh filename="package://manipulator_x_description/meshes/manipulator_x_link1.stl" scale="0.001 0.001 0.001"/>
@@ -73,5 +69,5 @@
     <parent link="link1"/>
     <child link="link2"/>
-    <origin xyz="0.012 0.0 0.034" rpy="0 0 0"/>
+    <origin xyz="0.048 0.0 0.137" rpy="0 0 0"/>
     <axis xyz="0 0 1"/>
     <limit velocity="6.5" effort="1000" lower="${-pi*0.9}" upper="${pi*0.9}" />
