Commit message: add gripper model

File: manipulator_x_description/urdf/manipulator_x.xacro (robot description, xacro)
@@ -273,5 +273,5 @@
   <joint name="joint6" type="revolute">
     <parent link="link6"/>
-    <child link="link789"/>
+    <child link="link7"/>
     <origin xyz="0.062 0.017 0.0" rpy="0 0 0"/>
     <axis xyz="1 0 0"/>
@@ -289,24 +289,106 @@
     </actuator>
   </transmission>
-  <!-- Link 789 -->
-  <link name="link789">
-    <collision>
-      <origin xyz="0 0 0" rpy="0 0 0"/>
-      <geometry>
-        <mesh filename="package://manipulator_x_description/meshes/manipulator_x_link789.stl" scale="0.001 0.001 0.001"/>
-      </geometry>
-    </collision>
-    <visual>
-      <origin xyz="0 0 0" rpy="0 0 0"/>
-      <geometry>
-        <mesh filename="package://manipulator_x_description/meshes/manipulator_x_link789.stl" scale="0.001 0.001 0.001"/>
-      </geometry>
-      <material name="grey"/>
-    </visual>
-    <inertial>
-      <origin xyz="0.04197 0.00146 -0.00021" rpy="0 0 0"/>
-      <mass value="0.26121"/>
-      <inertia ixx="1.0" ixy="0.0" ixz="0.0" iyy="1.0" iyz="0.0" izz="1.0" />
-      <!--<inertia ixx="0.00019" ixy="0.00001" ixz="0.0" iyy="0.00022" iyz="0.0" izz="0.00029" />-->
+  <!-- Link 7 -->
+  <link name="link7">
+    <collision>
+      <origin xyz="0 0 0" rpy="0 0 0"/>
+      <geometry>
+        <mesh filename="package://manipulator_x_description/meshes/manipulator_x_link7.stl" scale="0.001 0.001 0.001"/>
+      </geometry>
+    </collision>
+    <visual>
+      <origin xyz="0 0 0" rpy="0 0 0"/>
+      <geometry>
+        <mesh filename="package://manipulator_x_description/meshes/manipulator_x_link7.stl" scale="0.001 0.001 0.001"/>
+      </geometry>
+      <material name="grey"/>
+    </visual>
+    <inertial>
+      <origin xyz="0.02745 0.00300 -0.00043" rpy="0 0 0"/>
+      <mass value="0.12680"/>
+      <inertia ixx="1.0" ixy="0.0" ixz="0.0" iyy="1.0" iyz="0.0" izz="1.0" />
+      <!--<inertia ixx="0.00004897" ixy="-0.00000004" ixz="0.00000006" iyy="0.00003261" iyz="0.00000010" izz="0.00004008" />-->
+    </inertial>
+  </link>
+  <!-- Grip Joint -->
+  <joint name="grip_joint" type="revolute">
+    <parent link="link7"/>
+    <child link="grip_link"/>
+    <origin xyz="0.02900 -0.01600 0.02300" rpy="0 0 0"/>
+    <axis xyz="0 0 1"/>
+    <limit velocity="6.5" effort="1000" lower="${-0.5*pi}" upper="${0.5*pi}" />
+    <dynamics damping="0.7"/>
+  </joint>
+  <transmission name="tran7">
+    <type>transmission_interface/SimpleTransmission</type>
+    <joint name="grip_joint">
+      <hardwareInterface>EffortJointInterface</hardwareInterface>
+    </joint>
+    <actuator name="motor7">
+      <hardwareInterface>EffortJointInterface</hardwareInterface>
+      <mechanicalReduction>1</mechanicalReduction>
+    </actuator>
+  </transmission>
+  <!-- Grip Link -->
+  <link name="grip_link">
+    <collision>
+      <origin xyz="0 0 0" rpy="0 0 0"/>
+      <geometry>
+        <mesh filename="package://manipulator_x_description/meshes/manipulator_x_link9.stl" scale="0.001 0.001 0.001"/>
+      </geometry>
+    </collision>
+    <visual>
+      <origin xyz="0 0 0" rpy="0 0 0"/>
+      <geometry>
+        <mesh filename="package://manipulator_x_description/meshes/manipulator_x_link9.stl" scale="0.001 0.001 0.001"/>
+      </geometry>
+      <material name="grey"/>
+    </visual>
+    <inertial>
+      <origin xyz="0.02666 -0.00910 -0.02300" rpy="0 0 0"/>
+      <mass value="0.06721"/>
+      <inertia ixx="1.0" ixy="0.0" ixz="0.0" iyy="1.0" iyz="0.0" izz="1.0" />
+      <!--<inertia ixx="0.00002875" ixy="-0.00000593" ixz="-0.00000006" iyy="0.00006646" iyz="-0.00000009" izz="0.00005474" />-->
+    </inertial>
+  </link>
+  <!-- Grip Joint Sub -->
+  <joint name="grip_joint_sub" type="revolute">
+    <parent link="link7"/>
+    <child link="grip_link_sub"/>
+    <origin xyz="0.02900 0.01600 0.02300" rpy="0 0 0"/>
+    <axis xyz="0 0 -1"/>
+    <limit velocity="6.5" effort="1000" lower="${-0.5*pi}" upper="${0.5*pi}" />
+    <dynamics damping="0.7"/>
+  </joint>
+  <transmission name="tran8">
+    <type>transmission_interface/SimpleTransmission</type>
+    <joint name="grip_joint_sub">
+      <hardwareInterface>EffortJointInterface</hardwareInterface>
+    </joint>
+    <actuator name="motor8">
+      <hardwareInterface>EffortJointInterface</hardwareInterface>
+      <mechanicalReduction>1</mechanicalReduction>
+    </actuator>
+  </transmission>
+  <!-- Grip Link Sub -->
+  <link name="grip_link_sub">
+    <collision>
+      <origin xyz="0 0 0" rpy="0 0 0"/>
+      <geometry>
+        <mesh filename="package://manipulator_x_description/meshes/manipulator_x_link8.stl" scale="0.001 0.001 0.001"/>
+      </geometry>
+    </collision>
+    <visual>
+      <origin xyz="0 0 0" rpy="0 0 0"/>
+      <geometry>
+        <mesh filename="package://manipulator_x_description/meshes/manipulator_x_link8.stl" scale="0.001 0.001 0.001"/>
+      </geometry>
+      <material name="grey"/>
+    </visual>
+    <inertial>
+      <origin xyz="0.02666 0.00910 -0.02300" rpy="0 0 0"/>
+      <mass value="0.06721"/>
+      <inertia ixx="1.0" ixy="0.0" ixz="0.0" iyy="1.0" iyz="0.0" izz="1.0" />
+      <!--<inertia ixx="0.00002875" ixy="0.00000593" ixz="0.00000006" iyy="0.00006646" iyz="-0.00000009" izz="0.00005474" />-->
     </inertial>
   </link>

Commit message: mass property update

File: manipulator_x_description/urdf/manipulator_x.xacro (robot description, xacro)
@@ -42,4 +42,5 @@
     <parent link="base"/>
     <child link="link1"/>
+    <origin xyz="0.0 0.0 0.006" rpy="0 0 0"/>
   </joint>
   <!-- Link 1 -->
@@ -59,8 +60,8 @@
     </visual>
     <inertial>
-      <origin xyz="-0.01175 0.00000 -0.01620" rpy="0 0 0"/>
+      <origin xyz="0.00025 0.00000 0.01780" rpy="0 0 0"/>
       <mass value="0.08659"/>
       <inertia ixx="1.0" ixy="0.0" ixz="0.0" iyy="1.0" iyz="0.0" izz="1.0" />
-      <!--<inertia ixx="0.00000371" ixy="0.0" ixz="-0.00000025" iyy="0.00002369" iyz="0.0" izz="0.00002097" />-->
+      <!--<inertia ixx="0.00001371" ixy="0.0" ixz="-0.00000025" iyy="0.00002369" iyz="0.0" izz="0.00002097" />-->
     </inertial>
   </link>
@@ -69,5 +70,5 @@
     <parent link="link1"/>
     <child link="link2"/>
-    <origin xyz="0.0 0.0 0.042" rpy="0 0 0"/>
+    <origin xyz="0.012 0.0 0.036" rpy="0 0 0"/>
     <axis xyz="0 0 1"/>
     <limit velocity="6.5" effort="1000" lower="${-8.0*pi/9.0}" upper="${8.0*pi/9.0}" />
@@ -100,5 +101,5 @@
     </visual>
     <inertial>
-      <origin xyz="0.00000 0.00000 0.00975" rpy="0 0 0"/>
+      <origin xyz="0.00000 0.00000 0.00775" rpy="0 0 0"/>
       <mass value="0.00795"/>
       <inertia ixx="1.0" ixy="0.0" ixz="0.0" iyy="1.0" iyz="0.0" izz="1.0" />

Commit message: update

File: manipulator_x_description/urdf/manipulator_x.xacro (robot description, xacro)
@@ -20,58 +20,30 @@
   <link name="base">
     <collision>
-      <origin xyz="0 0 0" rpy="0 0 0"/>
-      <geometry>
-        <mesh filename="package://manipulator_x_description/meshes/manipulatorx7_rev1_base-plate.stl" scale="0.001 0.001 0.001"/>
-      </geometry>
-    </collision>
-    <visual>
-      <origin xyz="0 0 0" rpy="0 0 0"/>
-      <geometry>
-        <mesh filename="package://manipulator_x_description/meshes/manipulatorx7_rev1_base-plate.stl" scale="0.001 0.001 0.001"/>
-      </geometry>
-      <material name="grey"/>
-    </visual>
-    <inertial>
-      <origin xyz="0 0 0" rpy="0 0 0"/>
-      <mass value="1.0"/>
-      <inertia ixx="1.0" ixy="0.0" ixz="0" iyy="1.0" iyz="0.0" izz="1.0" />
-    </inertial>
-  </link>
-    <!-- Base fixed joint -->
-  <joint name="base_fixed" type="fixed">
-    <parent link="base"/>
-    <child link="link1"/>
-    <origin xyz="0.0 0.0 0.006" rpy="0 0 0"/>
-  </joint>
-  <!-- Link 1 -->
-  <link name="link1">
-    <collision>
-      <origin xyz="0 0 0" rpy="0 0 0"/>
-      <geometry>
-        <mesh filename="package://manipulator_x_description/meshes/manipulatorx7_rev1_axis-0.stl" scale="0.001 0.001 0.001"/>
-      </geometry>
-    </collision>
-    <visual>
-      <origin xyz="0 0 0" rpy="0 0 0"/>
-      <geometry>
-        <mesh filename="package://manipulator_x_description/meshes/manipulatorx7_rev1_axis-0.stl" scale="0.001 0.001 0.001"/>
-      </geometry>
-      <material name="grey"/>
-    </visual>
-    <inertial>
-      <origin xyz="0.00025 0.00000 0.01780" rpy="0 0 0"/>
-      <mass value="0.08659"/>
-      <inertia ixx="1.0" ixy="0.0" ixz="0.0" iyy="1.0" iyz="0.0" izz="1.0" />
-      <!--<inertia ixx="0.00001371" ixy="0.0" ixz="-0.00000025" iyy="0.00002369" iyz="0.0" izz="0.00002097" />-->
+      <origin xyz="0 0 0" rpy="0 0 ${-0.5*pi}"/>
+      <geometry>
+        <mesh filename="package://manipulator_x_description/meshes/assm_mpx540_6x_base.stl" scale="0.001 0.001 0.001"/>
+      </geometry>
+    </collision>
+    <visual>
+      <origin xyz="0 0 0" rpy="0 0 ${-0.5*pi}"/>
+      <geometry>
+        <mesh filename="package://manipulator_x_description/meshes/assm_mpx540_6x_base.stl" scale="0.001 0.001 0.001"/>
+      </geometry>
+      <material name="grey"/>
+    </visual>
+    <inertial>
+      <origin xyz="0 0 0" rpy="0 0 0"/>
+      <mass value="1.0"/>
+      <inertia ixx="1.0" ixy="0.0" ixz="0" iyy="1.0" iyz="0.0" izz="1.0" />
     </inertial>
   </link>
   <!-- Joint 1 -->
   <joint name="joint1" type="revolute">
-    <parent link="link1"/>
+    <parent link="base"/>
     <child link="link2"/>
-    <origin xyz="0.012 0.0 0.036" rpy="0 0 0"/>
+    <origin xyz="-0.021 0.0 0.023" rpy="0 0 0"/>
     <axis xyz="0 0 1"/>
     <limit velocity="6.5" effort="1000" lower="${-8.0*pi/9.0}" upper="${8.0*pi/9.0}" />
-    <dynamics damping="0.7"/>
+    <dynamics damping="0.1"/>
   </joint>
   <transmission name="tran1">
@@ -88,21 +60,20 @@
   <link name="link2">
     <collision>
-      <origin xyz="0 0 0" rpy="0 0 0"/>
-      <geometry>
-        <mesh filename="package://manipulator_x_description/meshes/manipulatorx7_rev1_axis-1.stl" scale="0.001 0.001 0.001"/>
-      </geometry>
-    </collision>
-    <visual>
-      <origin xyz="0 0 0" rpy="0 0 0"/>
-      <geometry>
-        <mesh filename="package://manipulator_x_description/meshes/manipulatorx7_rev1_axis-1.stl" scale="0.001 0.001 0.001"/>
-      </geometry>
-      <material name="grey"/>
-    </visual>
-    <inertial>
-      <origin xyz="0.00000 0.00000 0.00775" rpy="0 0 0"/>
-      <mass value="0.00795"/>
-      <inertia ixx="1.0" ixy="0.0" ixz="0.0" iyy="1.0" iyz="0.0" izz="1.0" />
-      <!--<inertia ixx="0.00000265" ixy="0.0" ixz="0.0" iyy="0.00000105" iyz="0.0" izz="0.00000246" />-->
+      <origin xyz="0 0 0" rpy="0 0 ${-0.5*pi}"/>
+      <geometry>
+        <mesh filename="package://manipulator_x_description/meshes/assm_mpx540_6x_0.stl" scale="0.001 0.001 0.001"/>
+      </geometry>
+    </collision>
+    <visual>
+      <origin xyz="0 0 0" rpy="0 0 ${-0.5*pi}"/>
+      <geometry>
+        <mesh filename="package://manipulator_x_description/meshes/assm_mpx540_6x_0.stl" scale="0.001 0.001 0.001"/>
+      </geometry>
+      <material name="grey"/>
+    </visual>
+    <inertial>
+      <origin xyz="0 0 0" rpy="0 0 0"/>
+      <mass value="1.0"/>
+      <inertia ixx="1.0" ixy="0.0" ixz="0" iyy="1.0" iyz="0.0" izz="1.0" />
     </inertial>
   </link>
@@ -111,8 +82,8 @@
     <parent link="link2"/>
     <child link="link3"/>
-    <origin xyz="0.0 -0.019 0.028" rpy="0 0 0"/>
+    <origin xyz="0.0 0.0 0.0495" rpy="0 0 0"/>
     <axis xyz="0 1 0"/>
-    <limit velocity="6.5" effort="1000" lower="${-pi*0.5}" upper="${pi*0.5}" />
-    <dynamics damping="0.7"/>
+    <limit velocity="6.5" effort="1000" lower="${-8.0*pi/9.0}" upper="${8.0*pi/9.0}" />
+    <dynamics damping="0.1"/>
   </joint>
   <transmission name="tran2">
@@ -129,21 +100,20 @@
   <link name="link3">
     <collision>
-      <origin xyz="0 0 0" rpy="0 0 0"/>
-      <geometry>
-        <mesh filename="package://manipulator_x_description/meshes/manipulatorx7_rev1_axis-2.stl" scale="0.001 0.001 0.001"/>
-      </geometry>
-    </collision>
-    <visual>
-      <origin xyz="0 0 0" rpy="0 0 0"/>
-      <geometry>
-        <mesh filename="package://manipulator_x_description/meshes/manipulatorx7_rev1_axis-2.stl" scale="0.001 0.001 0.001"/>
-      </geometry>
-      <material name="grey"/>
-    </visual>
-    <inertial>
-      <origin xyz="0.00000 0.01843 0.01319" rpy="0 0 0"/>
-      <mass value="0.09312"/>
-      <inertia ixx="1.0" ixy="0.0" ixz="0.0" iyy="1.0" iyz="0.0" izz="1.0" />
-      <!--<inertia ixx="0.0.00002889" ixy="0.0" ixz="0.0" iyy="0.0.00002519" iyz="-0.00000012" izz="0.00001549" />-->
+      <origin xyz="0 0 0" rpy="${-0.5*pi} 0 ${pi}"/>
+      <geometry>
+        <mesh filename="package://manipulator_x_description/meshes/assm_mpx540_6x_1.stl" scale="0.001 0.001 0.001"/>
+      </geometry>
+    </collision>
+    <visual>
+      <origin xyz="0 0 0" rpy="${-0.5*pi} 0 ${pi}"/>
+      <geometry>
+        <mesh filename="package://manipulator_x_description/meshes/assm_mpx540_6x_1.stl" scale="0.001 0.001 0.001"/>
+      </geometry>
+      <material name="grey"/>
+    </visual>
+    <inertial>
+      <origin xyz="0 0 0" rpy="0 0 0"/>
+      <mass value="1.0"/>
+      <inertia ixx="1.0" ixy="0.0" ixz="0" iyy="1.0" iyz="0.0" izz="1.0" />
     </inertial>
   </link>
@@ -152,8 +122,8 @@
     <parent link="link3"/>
     <child link="link4"/>
-    <origin xyz="0.0 0.019 0.0405" rpy="0 0 0"/>
-    <axis xyz="0 0 1"/>
-    <limit velocity="6.5" effort="1000" lower="${-8.0*pi/9.0}" upper="${8.0*pi/9.0}" />
-    <dynamics damping="0.7"/>
+    <origin xyz="0.029 0.0 0.102" rpy="0 0 0"/>
+    <axis xyz="0 1 0"/>
+    <limit velocity="6.5" effort="1000" lower="${-8.0*pi/9.0}" upper="${8.0*pi/9.0}" />
+    <dynamics damping="0.1"/>
   </joint>
   <transmission name="tran3">
@@ -170,21 +140,20 @@
   <link name="link4">
     <collision>
-      <origin xyz="0 0 0" rpy="0 0 0"/>
-      <geometry>
-        <mesh filename="package://manipulator_x_description/meshes/manipulatorx7_rev1_axis-3.stl" scale="0.001 0.001 0.001"/>
-      </geometry>
-    </collision>
-    <visual>
-      <origin xyz="0 0 0" rpy="0 0 0"/>
-      <geometry>
-        <mesh filename="package://manipulator_x_description/meshes/manipulatorx7_rev1_axis-3.stl" scale="0.001 0.001 0.001"/>
-      </geometry>
-      <material name="grey"/>
-    </visual>
-    <inertial>
-      <origin xyz="0.00024 -0.00036 0.04133" rpy="0 0 0"/>
-      <mass value="0.19398"/>
-      <inertia ixx="1.0" ixy="0.0" ixz="0.0" iyy="1.0" iyz="0.0" izz="1.0" />
-      <!--<inertia ixx="0.00012132" ixy="0.00000108" ixz="-0.00004800" iyy="0.00016807" iyz="0.00000157" izz="0.00007952" />-->
+      <origin xyz="0 0 0" rpy="0 0 ${-0.5*pi}"/>
+      <geometry>
+        <mesh filename="package://manipulator_x_description/meshes/assm_mpx540_6x_2.stl" scale="0.001 0.001 0.001"/>
+      </geometry>
+    </collision>
+    <visual>
+      <origin xyz="0 0 0" rpy="0 0 ${-0.5*pi}"/>
+      <geometry>
+        <mesh filename="package://manipulator_x_description/meshes/assm_mpx540_6x_2.stl" scale="0.001 0.001 0.001"/>
+      </geometry>
+      <material name="grey"/>
+    </visual>
+    <inertial>
+      <origin xyz="0 0 0" rpy="0 0 0"/>
+      <mass value="1.0"/>
+      <inertia ixx="1.0" ixy="0.0" ixz="0" iyy="1.0" iyz="0.0" izz="1.0" />
     </inertial>
   </link>
@@ -193,8 +162,8 @@
     <parent link="link4"/>
     <child link="link5"/>
-    <origin xyz="0.024 -0.019 0.064" rpy="0 0 0"/>
-    <axis xyz="0 -1 0"/>
-    <limit velocity="6.5" effort="1000" lower="${-pi*0.5}" upper="${pi*0.5}" />
-    <dynamics damping="0.7"/>
+    <origin xyz="0.045 0.0 0.024" rpy="0 0 0"/>
+    <axis xyz="1 0 0"/>
+    <limit velocity="6.5" effort="1000" lower="${-8.0*pi/9.0}" upper="${8.0*pi/9.0}" />
+    <dynamics damping="0.1"/>
   </joint>
   <transmission name="tran4">
@@ -211,21 +180,20 @@
   <link name="link5">
     <collision>
-      <origin xyz="0 0 0" rpy="0 0 0"/>
-      <geometry>
-        <mesh filename="package://manipulator_x_description/meshes/manipulatorx7_rev1_axis-4.stl" scale="0.001 0.001 0.001"/>
-      </geometry>
-    </collision>
-    <visual>
-      <origin xyz="0 0 0" rpy="0 0 0"/>
-      <geometry>
-        <mesh filename="package://manipulator_x_description/meshes/manipulatorx7_rev1_axis-4.stl" scale="0.001 0.001 0.001"/>
-      </geometry>
-      <material name="grey"/>
-    </visual>
-    <inertial>
-      <origin xyz="0.04301 0.01900 0.01187" rpy="0 0 0"/>
-      <mass value="0.09824"/>
-      <inertia ixx="1.0" ixy="0.0" ixz="0.0" iyy="1.0" iyz="0.0" izz="1.0" />
-      <!--<inertia ixx="0.00002597" ixy="0.0" ixz="-0.00000146" iyy="0.00003222" iyz="0.0" izz="0.00002303" />-->
+      <origin xyz="0 0 0" rpy="0 0 ${-0.5*pi}"/>
+      <geometry>
+        <mesh filename="package://manipulator_x_description/meshes/assm_mpx540_6x_3.stl" scale="0.001 0.001 0.001"/>
+      </geometry>
+    </collision>
+    <visual>
+      <origin xyz="0 0 0" rpy="0 0 ${-0.5*pi}"/>
+      <geometry>
+        <mesh filename="package://manipulator_x_description/meshes/assm_mpx540_6x_3.stl" scale="0.001 0.001 0.001"/>
+      </geometry>
+      <material name="grey"/>
+    </visual>
+    <inertial>
+      <origin xyz="0 0 0" rpy="0 0 0"/>
+      <mass value="1.0"/>
+      <inertia ixx="1.0" ixy="0.0" ixz="0" iyy="1.0" iyz="0.0" izz="1.0" />
     </inertial>
   </link>
@@ -234,8 +202,8 @@
     <parent link="link5"/>
     <child link="link6"/>
-    <origin xyz="0.064 0.019 0.024" rpy="0 0 0"/>
-    <axis xyz="1 0 0"/>
-    <limit velocity="6.5" effort="1000" lower="${-8.0*pi/9.0}" upper="${8.0*pi/9.0}" />
-    <dynamics damping="0.7"/>
+    <origin xyz="0.0595 0.0 0.0" rpy="0 0 0"/>
+    <axis xyz="0 1 0"/>
+    <limit velocity="6.5" effort="1000" lower="${-8.0*pi/9.0}" upper="${8.0*pi/9.0}" />
+    <dynamics damping="0.1"/>
   </joint>
   <transmission name="tran5">
@@ -252,21 +220,20 @@
   <link name="link6">
     <collision>
-      <origin xyz="0 0 0" rpy="0 0 0"/>
-      <geometry>
-        <mesh filename="package://manipulator_x_description/meshes/manipulatorx7_rev1_axis-5.stl" scale="0.001 0.001 0.001"/>
-      </geometry>
-    </collision>
-    <visual>
-      <origin xyz="0 0 0" rpy="0 0 0"/>
-      <geometry>
-        <mesh filename="package://manipulator_x_description/meshes/manipulatorx7_rev1_axis-5.stl" scale="0.001 0.001 0.001"/>
-      </geometry>
-      <material name="grey"/>
-    </visual>
-    <inertial>
-      <origin xyz="0.02731 -0.00057 0.00000" rpy="0 0 0"/>
-      <mass value="0.09312"/>
-      <inertia ixx="1.0" ixy="0.0" ixz="0.0" iyy="1.0" iyz="0.0" izz="1.0" />
-      <!--<inertia ixx="0.00001549" ixy="0.00000012" ixz="0.0" iyy="0.00002519" iyz="0.0" izz="0.00002889" />-->
+      <origin xyz="0 0 0" rpy="0 0 ${-0.5*pi}"/>
+      <geometry>
+        <mesh filename="package://manipulator_x_description/meshes/assm_mpx540_6x_4.stl" scale="0.001 0.001 0.001"/>
+      </geometry>
+    </collision>
+    <visual>
+      <origin xyz="0 0 0" rpy="0 0 ${-0.5*pi}"/>
+      <geometry>
+        <mesh filename="package://manipulator_x_description/meshes/assm_mpx540_6x_4.stl" scale="0.001 0.001 0.001"/>
+      </geometry>
+      <material name="grey"/>
+    </visual>
+    <inertial>
+      <origin xyz="0 0 0" rpy="0 0 0"/>
+      <mass value="1.0"/>
+      <inertia ixx="1.0" ixy="0.0" ixz="0" iyy="1.0" iyz="0.0" izz="1.0" />
     </inertial>
   </link>
@@ -275,8 +242,8 @@
     <parent link="link6"/>
     <child link="link7"/>
-    <origin xyz="0.0405 -0.019 0.0" rpy="0 0 0"/>
-    <axis xyz="0 -1 0"/>
-    <limit velocity="6.5" effort="1000" lower="${-pi*0.5}" upper="${pi*0.5}" />
-    <dynamics damping="0.7"/>
+    <origin xyz="0.045 0.0 0.0" rpy="0 0 0"/>
+    <axis xyz="1 0 0"/>
+    <limit velocity="6.5" effort="1000" lower="${-8.0*pi/9.0}" upper="${8.0*pi/9.0}" />
+    <dynamics damping="0.1"/>
   </joint>
   <transmission name="tran6">
@@ -293,144 +260,20 @@
   <link name="link7">
     <collision>
-      <origin xyz="0 0 0" rpy="0 0 0"/>
-      <geometry>
-        <mesh filename="package://manipulator_x_description/meshes/manipulatorx7_rev1_axis-6.stl" scale="0.001 0.001 0.001"/>
-      </geometry>
-    </collision>
-    <visual>
-      <origin xyz="0 0 0" rpy="0 0 0"/>
-      <geometry>
-        <mesh filename="package://manipulator_x_description/meshes/manipulatorx7_rev1_axis-6.stl" scale="0.001 0.001 0.001"/>
-      </geometry>
-      <material name="grey"/>
-    </visual>
-    <inertial>
-      <origin xyz="0.04301 0.01900 0.01142" rpy="0 0 0"/>
-      <mass value="0.09824"/>
-      <inertia ixx="1.0" ixy="0.0" ixz="0.0" iyy="1.0" iyz="0.0" izz="1.0" />
-      <!--<inertia ixx="0.00002594" ixy="0.0" ixz="-0.00000085" iyy="0.00003219" iyz="0.0" izz="0.00002303" />-->
-    </inertial>
-  </link>
-  <!-- Joint 7 -->
-  <joint name="joint7" type="revolute">
-    <parent link="link7"/>
-    <child link="link8"/>
-    <origin xyz="0.064 0.019 0.0" rpy="0 0 0"/>
-    <axis xyz="1 0 0"/>
-    <limit velocity="6.5" effort="1000" lower="${-8.0*pi/9.0}" upper="${8.0*pi/9.0}" />
-    <dynamics damping="0.7"/>
-  </joint>
-  <transmission name="tran7">
-    <type>transmission_interface/SimpleTransmission</type>
-    <joint name="joint7">
-      <hardwareInterface>EffortJointInterface</hardwareInterface>
-    </joint>
-    <actuator name="motor7">
-      <hardwareInterface>EffortJointInterface</hardwareInterface>
-      <mechanicalReduction>1</mechanicalReduction>
-    </actuator>
-  </transmission>
-  <!-- Link 8 -->
-  <link name="link8">
-    <collision>
-      <origin xyz="0 0 0" rpy="0 0 0"/>
-      <geometry>
-        <mesh filename="package://manipulator_x_description/meshes/manipulatorx7_rev1_axis-7.stl" scale="0.001 0.001 0.001"/>
-      </geometry>
-    </collision>
-    <visual>
-      <origin xyz="0 0 0" rpy="0 0 0"/>
-      <geometry>
-        <mesh filename="package://manipulator_x_description/meshes/manipulatorx7_rev1_axis-7.stl" scale="0.001 0.001 0.001"/>
-      </geometry>
-      <material name="grey"/>
-    </visual>
-    <inertial>
-      <origin xyz="0.02745 0.00300 -0.00043" rpy="0 0 0"/>
-      <mass value="0.12680"/>
-      <inertia ixx="1.0" ixy="0.0" ixz="0.0" iyy="1.0" iyz="0.0" izz="1.0" />
-      <!--<inertia ixx="0.00004897" ixy="-0.00000004" ixz="0.00000006" iyy="0.00003261" iyz="0.00000010" izz="0.00004008" />-->
-    </inertial>
-  </link>
-  <!-- Grip Joint -->
-  <joint name="grip_joint" type="revolute">
-    <parent link="link8"/>
-    <child link="grip_link"/>
-    <origin xyz="0.02900 -0.01600 0.02300" rpy="0 0 0"/>
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
Commit message: update

File: manipulator_x_description/urdf/manipulator_x.xacro (robot description, xacro)
@@ -123,5 +123,5 @@
     <child link="link4"/>
     <origin xyz="0.029 0.0 0.102" rpy="0 0 0"/>
-    <axis xyz="0 1 0"/>
+    <axis xyz="0 -1 0"/>
     <limit velocity="6.5" effort="1000" lower="${-8.0*pi/9.0}" upper="${8.0*pi/9.0}" />
     <dynamics damping="0.1"/>
@@ -203,5 +203,5 @@
     <child link="link6"/>
     <origin xyz="0.0595 0.0 0.0" rpy="0 0 0"/>
-    <axis xyz="0 1 0"/>
+    <axis xyz="0 -1 0"/>
     <limit velocity="6.5" effort="1000" lower="${-8.0*pi/9.0}" upper="${8.0*pi/9.0}" />
     <dynamics damping="0.1"/>
